Commit message: v1.0.0

File: src/test/fairino_moveit2_test/fr5_v6_robot/urdf/fr5_v6_robot.urdf (robot description, URDF)
Before this commit: robot fr5_v6_robot, 13 links, 12 joints
Links:
- added link tool_frame
Joints:
- added joint tool_joint: type fixed, parent wrist3_link, child tool_frame, origin xyz=0 0 0.15 rpy=0 0 0
